File: pcb/ESP_Heater.kicad_sch (KiCad schematic)
At the start: 17 parts

Commit message: added analog circuit for themostate and serial interface
Parts:
- added C? (x4): 0.1u, symbol Device:C
- added C?: 2.2u, symbol Device:C
- added C?: 10u, symbol Device:C
- added C?: 1u, symbol Device:C
- added ILED: Interface LED, symbol Device:LED
- added R? (x2): R, symbol Device:R
- added R?: 4.7k, symbol Device:R
- added R?: 12k, symbol Device:R
- added R?: 3.3k, symbol Device:R
- added TLED: Themostate LED, symbol Device:LED
- added U? (x2): LM358, symbol Amplifier_Operational:LM358
- added U?: AP2204K-5.0, Package_TO_SOT_SMD:SOT-23-5, symbol Regulator_Linear:AP2204K-5.0
- J?: value 7-8-9 Interface -> 7-8-9 Thermostate Interface
- PLED: renamed from D?; value PLED -> Power LED
Connections:
- net +3.3V: now also U?.1 (VDD1), U?.1 (VDD1), C?.1, C?.1
- net +5VA: now also U?.8 (VDD2), ILED.2 (A)
- net GND: now also U?.4 (GND1), U?.4 (GND1), C?.2, C?.2
- net at U?.6 (VOB): now also R?.2
- net +5VD: now reaches U?.8 (VDD2)
- net +5VD: now also C?.1, C?.1, TLED.2 (A), U?.5 (VOUT)
- net +24V: now reaches J?.1
- net +24V: now also C?.1, U?.1 (VIN), U?.3 (EN), U?.8 (V+)
- net at J?.3: now also R?.2, U?.1
- net GND2: now reaches J?.4
- net GND2: now also C?.2, C?.2, C?.2, C?.2, R?.1, R?.1, U?.2 (GND), U?.4 (V-)
- net GNDA renamed GND1
- net GND1: now also C?.2, R?.1
- new net: R?.2, TLED.1 (K)
- new net: C?.1, R?.1, U?.3 (+)
- new net: R?.1, R?.2, U?.2 (-)
- new net: ILED.1 (K), R?.2
Other:
- moved on the sheet: J?, U?
